File: ESD/Exp_8_FireAlarmMiniProj/EXP NO 8.kicad_pcb (KiCad board)
At the start: 2 copper layers, 57.3 x 20.9 mm, 6 parts, among them J1 Screw_Terminal_01x02, J2 Screw_Terminal_01x02, U1 LM741

Commit message: Update Eighth Exp in ESD
Parts:
- removed J2: Screw_Terminal_01x02, TerminalBlock_Phoenix:TerminalBlock_Phoenix_MKDS-1,5-2-5.08_1x02_P5.08mm_Horizontal
- added BZ1: Buzzer, Buzzer_Beeper:Buzzer_12x9.5RM7.6, F.Cu at (138.4, 73.7)
- added G***: LOGO, Desktop:logo1, F.Cu at (133.3, 83.7)
- added G***: LOGO, Desktop:logo1, F.Cu at (134.6, 83.7)
- added G***: LOGO, Desktop:eag, F.Cu at (116.3, 79.2)
- moved J1 1.17 mm to (101.7, 72.3)
Routing:
- net Net-(BZ1--): track 18.3 -> 12.8 mm
- net +9V: track 39.5 -> 44.0 mm
- net Net-(U1--): track 15.1 -> 17.4 mm
- net Net-(U1-+): track 19.7 -> 18.4 mm
Other:
- board size 57.3 x 20.9 mm -> 54.6 x 24.6 mm
- board text removed: "AAAC"
